File: KisonPill.sch (KiCad schematic (older format))
At the start: 39 parts, among them J1 USB_C_Receptacle_USB2.0, J2 Conn_01x19_Male, J3 Conn_01x19_Male, Q1 2N3904S-RTK/PS, Q2 2N3904S-RTK/PS, SW1 SW_Push, SW2 SW_Push, SW3 SW_DIP_x04, U1 CP2102N-A01-GQFN28, U2 ESP32-WROOM-32D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

Commit message: V4
Parts:
- removed U3: SPX1117M3-L-3-3/TR, Package_TO_SOT_SMD:SOT-223-3_TabPin2, symbol Regulator_Linear:AZ1117-3.3
- removed U4: ESP32FullConnector-KisonCommon, KisonCommon:jtag1.27-10, symbol KisonCommon:ESP32FullConnector
- added U3: XC6206P332MR, Package_TO_SOT_SMD:SOT-23, symbol Regulator_Linear:XC6206PxxxMR
- C3, C4: value 22uf -> 1uf; footprint Capacitor_SMD:C_1206_3216Metric -> Capacitor_SMD:C_0603_1608Metric; LCSC C319197 -> (none)
- Q1, Q2: value 2N3904S-RTK/PS -> S8050; LCSC C18536 -> (none)
- U7: symbol KisonCommon:ESP32FullConnector -> KisonCommon:ESP32FullConnectorRX
Connections:
- net +3V3: now also U7.10 (3V3), U3.2 (VO); no longer U7.7 (3V3)
- net EN: now also U7.4 (nRST); no longer U7.1 (TRST)
- net EXT_5V: now also U3.3 (VI)
- net FT2232RX: now also U7.2 (TX); no longer U7.9 (TX)
- net FT2232TX: now also U7.1 (RX); no longer U7.10 (RX)
- net GND: now also U7.9 (GND), U3.1 (GND); no longer U7.2 (GND)
- net IO0: now also U7.3 (IO0); no longer U7.8 (IO0)
- net IO12: now also U7.6 (TDI); no longer U7.3 (TDI)
- net IO13: now also U7.8 (TCLK); no longer U7.4 (TCLK)
- net IO15: now also U7.7 (TDO); no longer U7.6 (TDO)
Other:
- moved on the sheet: D5, R6

Commit message: V5
Fix BJT package bug :(
Parts:
- Q1, Q2: value S8050 -> SS8050; symbol Transistor_BJT:S8050 -> Transistor_BJT:2N3055; LCSC (none) -> C541705
Connections:
- net DTR: now also Q2.2 (E); no longer Q2.1 (E)
- net RTS: now also Q1.2 (E); no longer Q1.1 (E)
- net at R11.1: now also Q1.1 (B); no longer Q1.2 (B)
- net at R12.1: now also Q2.1 (B); no longer Q2.2 (B)
Other:
- note added: "Remember to double check the package\nof these BJTs.\nGot me twice already :("
Changed lines of the file:
@@
 $EndComp
 $Comp
-L Transistor_BJT:S8050 Q2
+L Transistor_BJT:2N3055 Q2
 U 1 1 60AFF185
 P 3000 1300
 F 0 "Q2" H 3190 1254 50  0000 L CNN
-F 1 "S8050" H 3190 1345 50  0000 L CNN
+F 1 "SS8050" H 3190 1345 50  0000 L CNN
 F 2 "Package_TO_SOT_SMD:SOT-23" H 3200 1225 50  0001 L CIN
 F 3 "http://www.unisonic.com.tw/datasheet/S8050.pdf" H 3000 1300 50  0001 L CNN
+F 4 "C541705" H 3000 1300 50  0001 C CNN "LCSC"
 	1    3000 1300
 	1    0    0    1
 $EndComp
 $Comp
-L Transistor_BJT:S8050 Q1
+L Transistor_BJT:2N3055 Q1
 U 1 1 60AFF79D
 P 3000 750
 F 0 "Q1" H 3190 796 50  0000 L CNN
-F 1 "S8050" H 3190 705 50  0000 L CNN
+F 1 "SS8050" H 3190 705 50  0000 L CNN
 F 2 "Package_TO_SOT_SMD:SOT-23" H 3200 675 50  0001 L CIN
 F 3 "http://www.unisonic.com.tw/datasheet/S8050.pdf" H 3000 750 50  0001 L CNN
+F 4 "C541705" H 3000 750 50  0001 C CNN "LCSC"
 	1    3000 750
 	1    0    0    -1
@@
 	740  4350 1180 4350
 Connection ~ 1180 4350
+Text Notes 3270 1100 0    50   ~ 0
+Remember to double check the package\nof these BJTs.\nGot me twice already :(
 $EndSCHEMATC
